Commit message: ur tf_prefix

File: ipa_demo_cell_description/urdf/ipa_demo_env.urdf.xacro (robot description, xacro)
@@ -4,5 +4,5 @@
      For more information, please see http://wiki.ros.org/sw_urdf_exporter -->
 <robot xmlns:xacro="http://wiki.ros.org/xacro">
-  <xacro:macro name="ipa_demo_env" params="prefix">
+  <xacro:macro name="ipa_demo_env" params="tf_prefix">
     <link name="env_link">
       <inertial>

File: ipa_demo_cell_description/urdf/ipa_ur_demo.urdf.xacro (robot description, xacro)
@@ -1,5 +1,5 @@
 <?xml version="1.0"?>
 <robot xmlns:xacro="http://ros.org/wiki/xacro" name="ur">
-  <xacro:arg name="prefix" default="" />
+  <xacro:arg name="tf_prefix" default="" />
   <xacro:arg name="name" default="ipa_ur_demo"/>
   <!-- Endeffector name -->
@@ -28,5 +28,5 @@
   <xacro:include filename="$(find ur_description)/urdf/ur_macro.xacro" />
   <xacro:ur_robot
-    prefix="$(arg prefix)"
+    tf_prefix="$(arg tf_prefix)"
     joint_limits_parameters_file="$(arg joint_limit_params)"
     kinematics_parameters_file="$(arg kinematics_params)"
@@ -40,9 +40,9 @@
     fake_sensor_commands="$(arg fake_sensor_commands)"
     headless_mode="$(arg headless_mode)"
-    initial_positions="${load_yaml(initial_positions_file)}" />
+    initial_positions="${xacro.load_yaml(initial_positions_file)}" />
   <!-- Include the cell and attach it to the world-->
   <xacro:include filename="$(find ipa_demo_cell_description)/urdf/ipa_demo_env.urdf.xacro" />
   <link name="world" />
-  <xacro:ipa_demo_env prefix="" />
+  <xacro:ipa_demo_env tf_prefix="" />
   <joint name="demo_env_joint" type="fixed">
     <parent link="world" />
@@ -58,5 +58,5 @@
   <!-- Sensor calibration -->
   <!-- Set the tcp according to Hand Eye Calibration-->
-  <xacro:property name="sensor_config" value="${load_yaml('$(arg calibration_config_file)')}" />
+  <xacro:property name="sensor_config" value="${xacro.load_yaml('$(arg calibration_config_file)')}" />
   <xacro:property name="tcp_sensor" value="${sensor_config['tcp_sensor']}"/>
   <link name="tcp_sensor_link" />
@@ -71,5 +71,5 @@
   </joint>
   <!-- Set the welding gun tool-->
-  <xacro:property name="welding_gun_config" value="${load_yaml('$(arg calibration_config_file)')}" />
+  <xacro:property name="welding_gun_config" value="${xacro.load_yaml('$(arg calibration_config_file)')}" />
   <xacro:property name="tcp_welding_gun" value="${welding_gun_config['tcp_welding_gun']}"/>
   <link name="tcp_welding_gun_link" />
@@ -85,5 +85,5 @@
   <!-- Attach the welding gun -->
   <xacro:include filename="$(find ipa_demo_cell_description)/urdf/$(arg endeffector).urdf.xacro" />
-  <xacro:endeffector prefix="" />
+  <xacro:endeffector tf_prefix="" />
   <xacro:property name="flange_welding_gun" value="${welding_gun_config['flange_welding_gun']}"/>
   <joint name="welding_gun_joint" type="fixed">

File: ipa_demo_cell_description/urdf/welding_gun_lorch_scancontrol_3000.urdf.xacro (robot description, xacro)
@@ -4,5 +4,5 @@
      For more information, please see http://wiki.ros.org/sw_urdf_exporter -->
 <robot xmlns:xacro="http://wiki.ros.org/xacro">
-  <xacro:macro name="endeffector" params="prefix">
+  <xacro:macro name="endeffector" params="tf_prefix">
     <link name="welding_gun_link">
       <inertial>

File: ipa_moveit_config/srdf/ur.srdf.xacro (robot description, xacro)
@@ -4,6 +4,6 @@
   <xacro:arg name="name" default="ur"/>
   <!-- parameters -->
-  <xacro:arg name="prefix" default="" />
+  <xacro:arg name="tf_prefix" default="" />
   <xacro:include filename="$(find ipa_moveit_config)/srdf/ur_macro.srdf.xacro"/>
-  <xacro:ur_srdf name="$(arg name)" prefix="$(arg prefix)"/>
+  <xacro:ur_srdf name="$(arg name)" tf_prefix="$(arg tf_prefix)"/>
 </robot>

File: ipa_moveit_config/srdf/ur_macro.srdf.xacro (robot description, xacro)
@@ -5,5 +5,5 @@
     A URDF file must exist for this robot as well, where the joints and the links that are referenced are defined
 -->
-  <xacro:macro name="ur_srdf" params="name prefix">
+  <xacro:macro name="ur_srdf" params="name tf_prefix">
     <!--GROUPS - Representation of a set of joints and links. This can be useful for specifying DOF to plan for, defining arms, end effectors, etc-->
     <!--LINKS - When a link is specified, the parent joint of that link (if it exists) is automatically included-->
@@ -11,6 +11,6 @@
     <!--CHAINS - When a chain is specified, all the links along the chain (including endpoints) are included in the group. Additionally, all the joints that are parents to included links are also included. This means that joints along the chain and the parent joint of the base link are included in the group-->
     <!--SUBGROUPS - Groups can also be formed by referencing to already defined group names-->
-    <group name="${prefix}${name}_manipulator">
-      <chain base_link="${prefix}base_link" tip_link="tcp_welding_gun_link" />
+    <group name="${tf_prefix}${name}_manipulator">
+      <chain base_link="${tf_prefix}base_link" tip_link="tcp_welding_gun_link" />
     </group>
     <group name="welding_gun">
@@ -18,53 +18,53 @@
     </group>
     <!--GROUP STATES - Purpose - Define a named state for a particular group, in terms of joint values. This is useful to define states like 'folded arms'-->
-    <group_state name="${prefix}home" group="${prefix}${name}_manipulator">
-      <joint name="${prefix}elbow_joint" value="0" />
-      <joint name="${prefix}shoulder_lift_joint" value="-1.5707" />
-      <joint name="${prefix}shoulder_pan_joint" value="0" />
-      <joint name="${prefix}wrist_1_joint" value="0" />
-      <joint name="${prefix}wrist_2_joint" value="0" />
-      <joint name="${prefix}wrist_3_joint" value="0" />
+    <group_state name="${tf_prefix}home" group="${tf_prefix}${name}_manipulator">
+      <joint name="${tf_prefix}elbow_joint" value="0" />
+      <joint name="${tf_prefix}shoulder_lift_joint" value="-1.5707" />
+      <joint name="${tf_prefix}shoulder_pan_joint" value="0" />
+      <joint name="${tf_prefix}wrist_1_joint" value="0" />
+      <joint name="${tf_prefix}wrist_2_joint" value="0" />
+      <joint name="${tf_prefix}wrist_3_joint" value="0" />
     </group_state>
-    <group_state name="${prefix}up" group="${prefix}${name}_manipulator">
-      <joint name="${prefix}elbow_joint" value="0" />
-      <joint name="${prefix}shoulder_lift_joint" value="-1.5707" />
-      <joint name="${prefix}shoulder_pan_joint" value="0" />
-      <joint name="${prefix}wrist_1_joint" value="-1.5707" />
-      <joint name="${prefix}wrist_2_joint" value="0" />
-      <joint name="${prefix}wrist_3_joint" value="0" />
+    <group_state name="${tf_prefix}up" group="${tf_prefix}${name}_manipulator">
+      <joint name="${tf_prefix}elbow_joint" value="0" />
+      <joint name="${tf_prefix}shoulder_lift_joint" value="-1.5707" />
+      <joint name="${tf_prefix}shoulder_pan_joint" value="0" />
+      <joint name="${tf_prefix}wrist_1_joint" value="-1.5707" />
+      <joint name="${tf_prefix}wrist_2_joint" value="0" />
+      <joint name="${tf_prefix}wrist_3_joint" value="0" />
     </group_state>
-    <group_state name="${prefix}test_configuration" group="${prefix}${name}_manipulator">
-      <joint name="${prefix}elbow_joint" value="1.4" />
-      <joint name="${prefix}shoulder_lift_joint" value="-1.62" />
-      <joint name="${prefix}shoulder_pan_joint" value="1.54" />
-      <joint name="${prefix}wrist_1_joint" value="-1.2" />
-      <joint name="${prefix}wrist_2_joint" value="-1.6" />
-      <joint name="${prefix}wrist_3_joint" value="-0.11" />
+    <group_state name="${tf_prefix}test_configuration" group="${tf_prefix}${name}_manipulator">
+      <joint name="${tf_prefix}elbow_joint" value="1.4" />
+      <joint name="${tf_prefix}shoulder_lift_joint" value="-1.62" />
+      <joint name="${tf_prefix}shoulder_pan_joint" value="1.54" />
+      <joint name="${tf_prefix}wrist_1_joint" value="-1.2" />
+      <joint name="${tf_prefix}wrist_2_joint" value="-1.6" />
+      <joint name="${tf_prefix}wrist_3_joint" value="-0.11" />
     </group_state>
-    <group_state name="${prefix}pre_welding_configuration" group="${prefix}${name}_manipulator">
-      <joint name="${prefix}elbow_joint" value="2.22" />
-      <joint name="${prefix}shoulder_lift_joint" value="-1.93" />
-      <joint name="${prefix}shoulder_pan_joint" value="0.86" />
-      <joint name="${prefix}wrist_1_joint" value="-1.97" />
-      <joint name="${prefix}wrist_2_joint" value="-1.63" />
-      <joint name="${prefix}wrist_3_joint" value="0.72" />
+    <group_state name="${tf_prefix}pre_welding_configuration" group="${tf_prefix}${name}_manipulator">
+      <joint name="${tf_prefix}elbow_joint" value="2.22" />
+      <joint name="${tf_prefix}shoulder_lift_joint" value="-1.93" />
+      <joint name="${tf_prefix}shoulder_pan_joint" value="0.86" />
+      <joint name="${tf_prefix}wrist_1_joint" value="-1.97" />
+      <joint name="${tf_prefix}wrist_2_joint" value="-1.63" />
+      <joint name="${tf_prefix}wrist_3_joint" value="0.72" />
     </group_state>
     <!--END EFFECTOR - Purpose - Represent information about an end effector.-->
     <end_effector name="welding_ee" parent_link="tcp_welding_gun_link" group="welding_gun" />
     <!--VIRTUAL JOINT - Purpose - this element defines a virtual joint between a robot link and an external frame of reference (considered fixed with respect to the robot)-->
-    <joint name="${prefix}fixed_base" type="fixed" parent_frame="world" child_link="${prefix}base_link" />
+    <joint name="${tf_prefix}fixed_base" type="fixed" parent_frame="world" child_link="${tf_prefix}base_link" />
     <!--DISABLE COLLISIONS - By default it is assumed that any link of the robot could potentially come into collision with any other link in the robot. This tag disables collision checking between a specified pair of links. -->
-    <disable_collisions link1="${prefix}base_link" link2="${prefix}base_link_inertia" reason="Adjacent" />
-    <disable_collisions link1="${prefix}base_link_inertia" link2="${prefix}shoulder_link" reason="Adjacent" />
-    <disable_collisions link1="${prefix}tool0" link2="${prefix}wrist_1_link" reason="Never" />
-    <disable_collisions link1="${prefix}tool0" link2="${prefix}wrist_2_link" reason="Never" />
-    <disable_collisions link1="${prefix}tool0" link2="${prefix}wrist_3_link" reason="Adjacent" />
-    <disable_collisions link1="${prefix}forearm_link" link2="${prefix}upper_arm_link" reason="Adjacent" />
-    <disable_collisions link1="${prefix}forearm_link" link2="${prefix}wrist_1_link" reason="Adjacent" />
-    <disable_collisions link1="${prefix}shoulder_link" link2="${prefix}upper_arm_link" reason="Adjacent" />
-    <disable_collisions link1="${prefix}wrist_1_link" link2="${prefix}wrist_2_link" reason="Adjacent" />
-    <disable_collisions link1="${prefix}wrist_1_link" link2="${prefix}wrist_3_link" reason="Never" />
-    <disable_collisions link1="${prefix}wrist_2_link" link2="${prefix}wrist_3_link" reason="Adjacent" />
-    <disable_collisions link1="welding_gun_link" link2="${prefix}wrist_3_link" reason="Adjacent" />
+    <disable_collisions link1="${tf_prefix}base_link" link2="${tf_prefix}base_link_inertia" reason="Adjacent" />
+    <disable_collisions link1="${tf_prefix}base_link_inertia" link2="${tf_prefix}shoulder_link" reason="Adjacent" />
+    <disable_collisions link1="${tf_prefix}tool0" link2="${tf_prefix}wrist_1_link" reason="Never" />
+    <disable_collisions link1="${tf_prefix}tool0" link2="${tf_prefix}wrist_2_link" reason="Never" />
+    <disable_collisions link1="${tf_prefix}tool0" link2="${tf_prefix}wrist_3_link" reason="Adjacent" />
+    <disable_collisions link1="${tf_prefix}forearm_link" link2="${tf_prefix}upper_arm_link" reason="Adjacent" />
+    <disable_collisions link1="${tf_prefix}forearm_link" link2="${tf_prefix}wrist_1_link" reason="Adjacent" />
+    <disable_collisions link1="${tf_prefix}shoulder_link" link2="${tf_prefix}upper_arm_link" reason="Adjacent" />
+    <disable_collisions link1="${tf_prefix}wrist_1_link" link2="${tf_prefix}wrist_2_link" reason="Adjacent" />
+    <disable_collisions link1="${tf_prefix}wrist_1_link" link2="${tf_prefix}wrist_3_link" reason="Never" />
+    <disable_collisions link1="${tf_prefix}wrist_2_link" link2="${tf_prefix}wrist_3_link" reason="Adjacent" />
+    <disable_collisions link1="welding_gun_link" link2="${tf_prefix}wrist_3_link" reason="Adjacent" />
     <disable_collisions link1="base_link_inertia" link2="env_link" reason="Adjacent" />
   </xacro:macro>
